File: untitled.kicad_sch (KiCad schematic)
At the start: 8 parts, among them J1 Conn_01x08, U1 ADS131M08QPBSRQ1, Y2 Crystal!

Commit message: rough layout done -connectors are not fully chosen yet, nano for temp, ??? for volt taps
Parts:
- removed J1: Conn_01x08, symbol Connector_Generic:Conn_01x08
- removed Y2: Crystal!, symbol Device:Crystal_Small
- added C14, C15, C16, C17, C18: 4.7nF, Capacitor_SMD:C_0805_2012Metric, symbol Device:C_Small
- added C19, C20: 36pF, Capacitor_SMD:C_0805_2012Metric, symbol Device:C_Small
- added J3: temptap0, Connector_Molex:Molex_Micro-Fit_3.0_43650-0400_1x04_P3.00mm_Horizontal, symbol Connector_Generic:Conn_01x04
- added J7: temptap1, Connector_Molex:Molex_Micro-Fit_3.0_43650-0400_1x04_P3.00mm_Horizontal, symbol Connector_Generic:Conn_01x04
- added J8: extratemp1, Connector_Molex:Molex_Micro-Fit_3.0_43650-0200_1x02_P3.00mm_Horizontal, symbol Connector_Generic:Conn_01x02
- added J9: extratemp2, Connector_Molex:Molex_Micro-Fit_3.0_43650-0200_1x02_P3.00mm_Horizontal, symbol Connector_Generic:Conn_01x02
- added R16, R17, R18, R19, R20, R21: 50Ω, Resistor_SMD:R_0805_2012Metric, symbol Device:R
- added XTAL1: ABM3-8.000MHZ-D2Y-T, XTAL_ABM3-8.000MHZ-D2Y-T_ABR, symbol ABM3 - 8mhz:ABM3-8.000MHZ-D2Y-T
- C1, C2, C3: footprint (none) -> Capacitor_SMD:C_0805_2012Metric
- R1, R2: footprint (none) -> Resistor_SMD:R_0805_2012Metric
- U1: footprint TQFP32_PBS_TEX -> footprints:TQFP32_PBS_TEX
Connections:
- net AIN6 is gone; now on net GNDA: U1.9 (AIN6P)
- net AIN7 is gone; now on net GNDA: U1.12 (AIN7P)
- net AIN0: now also C16.1, R20.1
- net AIN1: now also C16.2, C17.1, R19.1
- net AIN2: now also C15.1, C17.2, R18.1
- net AIN3: now also C14.1, C15.2, R16.1
- net AIN4: now also C14.2, C18.1, R17.1
- net AIN5: now also C18.2, R21.1
- net GNDA: now also J3.1 (Pin_1), J3.3 (Pin_3), J7.1 (Pin_1), J7.3 (Pin_3), J8.1 (Pin_1), J9.1 (Pin_1)
- net xtal2: now reaches U1.22 (XTAL2)
- net xtal2: now also C19.2
- net xtal1: now reaches U1.23 (XTAL1/CLKIN)
- net xtal1: now also C20.2
- new net: C19.1, XTAL1.1
- new net: C20.1, XTAL1.2
- new net temp0: J3.4 (Pin_4), R20.2
- new net temp1: J3.2 (Pin_2), R19.2
- new net temp2: J7.4 (Pin_4), R18.2
- new net temp3: J7.2 (Pin_2), R16.2
- new net temp4: J9.2 (Pin_2), R17.2
- new net temp5: J8.2 (Pin_2), R21.2
Other:
- note added: "Temperature taps"
- moved on the sheet: C1, C2, C3, R1, R2, U1
