File: ADC_related.kicad_sch (KiCad schematic)
At the start: 24 parts, among them J3 temptap0, J7 temptap1, J8 extratemp1, J9 extratemp2, U1 ADS131M08QPBSRQ1

Commit message: Addressed some concerns
Parts:
- added J6: Conn_01x05_Pin, symbol Connector:Conn_01x05_Pin
- added SW3: SW_DIP_x02, symbol Switch:SW_DIP_x02
- added TP15, TP16: TestPoint_Small, symbol Connector:TestPoint_Small
- added TP8: Temp2test, symbol Connector:TestPoint_Small
- added TP9: Temp0test, symbol Connector:TestPoint_Small
Connections:
- net CS: now also J6.5 (Pin_5)
- net DRDY: now also J6.4 (Pin_4)
- net MISO: now also J6.2 (Pin_2)
- net MOSI: now also J6.1 (Pin_1)
- net SCLK: now also J6.3 (Pin_3)
- net temp0: now also SW3.4, TP15.1; no longer J3.4 (Pin_4)
- net temp1: now also SW3.3, TP16.1; no longer J3.2 (Pin_2)
- net temp2: now also TP8.1
- new net: J3.4 (Pin_4), SW3.1, TP9.1
- new net: J3.2 (Pin_2), SW3.2
Other:
- note added: "Temperature tap Antialiasing"
- note added: "scrutineering temp inject"
- note added: "standard LHR solar crystal"
- note added: "test points for SPI"
- moved on the sheet: C14, C15, C16, C17, C18, J3, J8, J9, R16, R17, R18, R19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
