File: hardware/VoltTemp/TemperatureFilter.kicad_sch (KiCad schematic)
At the start: 9 parts

Commit message: more progress on schematic
Parts:
- removed U (x3): Opamp_Dual, symbol Device:Opamp_Dual
- added U7: Opamp_Dual, symbol Device:Opamp_Dual
- renumbered C to C32, R to R49
Connections:
- net GNDA: now also U7.4 (V-)
- net VDDA: now also U7.8 (V+)
- net tempIn: now also U7.3 (+)
- net tempOut: now also U7.7
- net at R49.1: now also U7.1, U7.2 (-)
- net at C25.1, C32.1, R34.2: now also U7.5 (+)
- net at R35.2, R36.1: now also U7.6 (-)
