File: hardware/VoltTemp/TemperatureFilters.kicad_sch (KiCad schematic)
At the start: 0 parts

Commit message: progress
Other:
- added sheet TemperatureFilter0 (TemperatureFilter.kicad_sch)
- added sheet TemperatureFilter1 (TemperatureFilter.kicad_sch)
- added sheet TemperatureFilter2 (TemperatureFilter.kicad_sch)
- added sheet TemperatureFilter3 (TemperatureFilter.kicad_sch)
- added sheet TemperatureFilter4 (TemperatureFilter.kicad_sch)

Commit message: more progress on schematic
Changed lines of the file:
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@@
 		)
 	)
-	(hierarchical_label "Temperatures[0..4]"
+	(hierarchical_label "Temperature[0..4]"
 		(shape output)
 		(at 154.94 60.96 0)
