File: hardware/VoltTemp/TemperatureConn.kicad_sch (KiCad schematic)
At the start: 0 parts

Commit message: more progress on schematic
Parts:
- added J15: Conn_01x07, symbol Connector_Generic:Conn_01x07
Connections:
- net rawTemperature0: now also J15.6 (Pin_6)
- net rawTemperature1: now also J15.5 (Pin_5)
- net rawTemperature2: now also J15.4 (Pin_4)
- net rawTemperature3: now also J15.3 (Pin_3)
- net rawTemperature4: now also J15.2 (Pin_2)
- new net GNDA: J15.7 (Pin_7)
- new net VDDA: J15.1 (Pin_1)

Commit message: add scrutineering stuff
Parts:
- added J6: Conn_01x04, symbol Connector_Generic:Conn_01x04
- added R24: 0Ω, Resistor_SMD:R_0805_2012Metric, symbol Device:R
Connections:
- net GNDA: now also J6.4 (Pin_4)
- net VDDA: now also J6.1 (Pin_1)
- net rawTemperature1: now also J6.2 (Pin_2), R24.1; no longer J15.5 (Pin_5)
- new net rawTemperature1_Pre: J15.5 (Pin_5), J6.3 (Pin_3), R24.2
Other:
- note added: "For scrutineering we're routing one thermistor output to scrut board That output will be disconnected by scrut board and a new signal injected"
- note added: "Only one of 8 volttemps will connect to scrut Other volttemps will have 0 ohm bypass"
- note added: "Temperature Scrutineering"
