File: hardware/VoltTemp/VoltageConn.kicad_sch (KiCad schematic)
At the start: 45 parts, among them J1 VoltTap2, J2 VoltTap1

Commit message: more progress on schematic
Parts:
- removed F1, F2, F3, F4, F5: 10mA, UTSVT_Special:ptc_fuse_FUSC1607X75N, symbol Device:Polyfuse_Small
- removed F6: 40mA, UTSVT_Special:ptc_fuse_FUSC1607X75N, symbol Device:Polyfuse_Small
- removed J1: VoltTap2, Connector_Molex:Molex_Nano-Fit_105313-xx05_1x05_P2.50mm_Horizontal, symbol Connector_Generic:Conn_01x05
- removed J2: VoltTap1, Connector_Molex:Molex_Nano-Fit_105313-xx05_1x05_P2.50mm_Horizontal, symbol Connector_Generic:Conn_01x05
- removed S1: 418121270806, footprints:418121270806, symbol 418121270806:418121270806
- removed TP10: 4&5inject, TestPoint:TestPoint_Keystone_5010-5014_Multipurpose, symbol Connector:TestPoint_Small
- removed TP11: 3&4inject, TestPoint:TestPoint_Keystone_5010-5014_Multipurpose, symbol Connector:TestPoint_Small
- removed TP12: 2&3inject, TestPoint:TestPoint_Keystone_5010-5014_Multipurpose, symbol Connector:TestPoint_Small
- removed TP13: 1&2inject, TestPoint:TestPoint_Keystone_5010-5014_Multipurpose, symbol Connector:TestPoint_Small
- removed TP14: cellgndinject, TestPoint:TestPoint_Keystone_5010-5014_Multipurpose, symbol Connector:TestPoint_Small
- removed TP2: last_cell, UTSVT_Special:TestPoint_HEX_3mmID, symbol Connector:TestPoint_Small
- removed TP3: 4&5 COM, UTSVT_Special:TestPoint_HEX_3mmID, symbol Connector:TestPoint_Small
- removed TP4: 3&4 COM, UTSVT_Special:TestPoint_HEX_3mmID, symbol Connector:TestPoint_Small
- removed TP5: 2&3 COM, UTSVT_Special:TestPoint_HEX_3mmID, symbol Connector:TestPoint_Small
- removed TP6: 1&2 COM, UTSVT_Special:TestPoint_HEX_3mmID, symbol Connector:TestPoint_Small
- removed TP7: GND2, UTSVT_Special:TestPoint_HEX_3mmID, symbol Connector:TestPoint_Small
- removed TP9: last_inject, TestPoint:TestPoint_Keystone_5010-5014_Multipurpose, symbol Connector:TestPoint_Small
- added J1: Conn_01x11, symbol Connector_Generic:Conn_01x11
Connections:
- net at F10.1: now also J1.7 (Pin_7)
- net at F8.1: now also J1.3 (Pin_3)
- net at F7.1: now also J1.1 (Pin_1)
- net at F9.1: now also J1.5 (Pin_5)
- net at F11.1: now also J1.9 (Pin_9)
- net at F12.1: now also J1.11 (Pin_11)
- no-connect marks 4 -> 5
Other:
- note added: "Voltage taps are fused at 10mA by regs GND2 is fused at a higher current (40mA)"
- note removed: "Using two connectors allows us to use different cell configurations if desired. It also allows us to use nano-fit connectors."
- note removed: "Voltage taps (DIP switch for scrutineering)"
- moved on the sheet: F10, F11, F12, F7, F8, F9

Commit message: add scrutineering stuff
Parts:
- removed R11: 0Ω, Resistor_SMD:R_0805_2012Metric, symbol Device:R
- added J7: Conn_01x04, symbol Connector_Generic:Conn_01x04
- added R23: 0Ω, Resistor_SMD:R_0805_2012Metric, symbol Device:R
Connections:
- net 3&4COM: now also J7.1 (Pin_1), R23.1; no longer R19.2
- net GND2: now also J7.4 (Pin_4)
- new net 3&4COM_Out: J7.3 (Pin_3), R19.2, R23.2
- no-connect marks 5 -> 6
Other:
- note added: "For voltage scrutineering we will pass one tap to the scrut board that tap will be disconnected for scrutineering and a new signal injected that tap will be routed back to this volttemp"
- note added: "Voltage Connector"
- note added: "Voltage Scrutineering"
- note removed: "volt tap antialiasing"
- moved on the sheet: C10, C11, C6, C7, C8, C9, R12, R13, R14, R15, R16, R17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
