File: PS-CellSim/PS-CellSim.kicad_pcb (KiCad board)
At the start: 2 copper layers, 49.7 x 59.8 mm, 57 parts, among them J1 bms_taps, J2 bench_vcc, J3 bench_gnd, J4 bms_ref, J5 bms_gpio_set2, J6 bms_gpio_set1, J7 therm_set1, J8 therm_set2

Commit message: layour layouted
Parts:
- added 1&2: TestPoint, TestPoint:TestPoint_Plated_Hole_D2.0mm, F.Cu at (128.4, 63.3)
- added 2&3: TestPoint, TestPoint:TestPoint_Plated_Hole_D2.0mm, F.Cu at (133.7, 63.3)
- added 28.8[v]: TestPoint, TestPoint:TestPoint_Plated_Hole_D2.0mm, F.Cu at (165.1, 63.3)
- added 3&4: TestPoint, TestPoint:TestPoint_Plated_Hole_D2.0mm, F.Cu at (138.9, 63.3)
- added 4&5: TestPoint, TestPoint:TestPoint_Plated_Hole_D2.0mm, F.Cu at (144.1, 63.3)
- added 5&6: TestPoint, TestPoint:TestPoint_Plated_Hole_D2.0mm, F.Cu at (149.4, 63.3)
- added 6&7: TestPoint, TestPoint:TestPoint_Plated_Hole_D2.0mm, F.Cu at (154.6, 63.3)
- added 7&8: TestPoint, TestPoint:TestPoint_Plated_Hole_D2.0mm, F.Cu at (159.8, 63.3)
- added GND: TestPoint, TestPoint:TestPoint_Plated_Hole_D2.0mm, F.Cu at (123.2, 63.3)
- moved JP1 5.26 mm to (131.8, 66.9)
- moved JP2 5.26 mm to (135.3, 66.9)
- moved JP3 5.26 mm to (138.8, 66.9)
- moved JP4 5.26 mm to (142.2, 66.9)
- moved JP5 5.26 mm to (145.7, 66.9)
- moved JP6 5.26 mm to (149.2, 66.9)
- moved JP7 5.26 mm to (152.6, 66.9)
- moved JP8 5.26 mm to (156.1, 66.9)
- moved J1 5.26 mm to (151.5, 72.4)
- moved J2 5.26 mm to (162.0, 76.5)
- moved J3 5.26 mm to (126.1, 76.4)
- moved R1 5.26 mm to (131.8, 69.0)
- moved R2 5.26 mm to (135.3, 69.0)
- moved R3 5.26 mm to (138.8, 69.0)
- moved R4 5.26 mm to (142.3, 69.0)
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Routing:
- net VCC: track 11.7 -> 21.5 mm
- net GND: track 11.6 -> 21.0 mm
- net /7&8: track 10.9 -> 17.3 mm
- net /1&2: track 11.1 -> 17.4 mm
- net /6&7: track 10.8 -> 15.5 mm
- net /2&3: track 10.5 -> 15.1 mm
- net /4&5: track 10.4 -> 14.5 mm
- net /5&6: track 10.2 -> 14.2 mm
- net /3&4: track 10.9 -> 14.8 mm
- net GND1: track 11.6 -> 12.4 mm
Other:
- board size 49.7 x 59.8 mm -> 49.9 x 64.5 mm
- board text added: "1"
- board text added: "2"
- board text added: "28.8[v]"
- board text added: "3"
- board text added: "4"
- board text added: "5"
- board text added: "6"
- board text added: "7"
- board text added: "8"
- board text added: "GND"
- board text added: "GPIO ->"
- board text added: "THERMISTORS"
- board text added: "TSREF BMSGND"
- board text added: "gnd"

Commit message: now has kicad sharepoint smiley face :)
Parts:
- J1: footprint UTSVT_Connectors:Molex_Nano-Fit_105313-xx07_1x07_P2.50mm_Horizontal -> LHRS_Connectors:Molex_Nano-Fit_105313-xx07_1x07_P2.50mm_Horizontal
- J2, J3: footprint UTSVT_Connectors:Banana_Jack_1_Pin_4mm -> LHRS_Connectors:Banana_Jack_1_Pin_4mm
- J4: footprint UTSVT_Connectors:Molex_Nano-Fit_105313-xx02_1x02_P2.50mm_Horizontal -> LHRS_Connectors:Molex_Nano-Fit_105313-xx02_1x02_P2.50mm_Horizontal
- J5, J6: footprint UTSVT_Connectors:Molex_Nano-Fit_105313-xx04_1x04_P2.50mm_Horizontal -> LHRS_Connectors:Molex_Nano-Fit_105313-xx04_1x04_P2.50mm_Horizontal
- J7, J8: footprint UTSVT_Connectors:Molex_Nano-Fit_105313-xx05_1x05_P2.50mm_Horizontal -> LHRS_Connectors:Molex_Nano-Fit_105313-xx05_1x05_P2.50mm_Horizontal
- renumbered GND to TP1, 1&2 to TP2, 2&3 to TP3, 3&4 to TP4, 4&5 to TP5, 5&6 to TP6, 6&7 to TP7, 7&8 to TP8, 28.8[v] to TP9
Changed lines of the file:
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@@
 		(embedded_fonts no)
 	)
-	(footprint "UTSVT_Connectors:Molex_Nano-Fit_105313-xx02_1x02_P2.50mm_Horizontal"
+	(footprint "LHRS_Connectors:Molex_Nano-Fit_105313-xx02_1x02_P2.50mm_Horizontal"
 		(layer "F.Cu")
 		(at 158 53.575)
@@
 		(descr "Plated Hole as test Point, diameter 2.0mm")
 		(tags "test point plated hole")
-		(property "Reference" "4&5"
+		(property "Reference" "TP5"
 			(at 0 -2.498 0)
 			(layer "F.SilkS")
@@
 		(embedded_fonts no)
 	)
-	(footprint "UTSVT_Connectors:Banana_Jack_1_Pin_4mm"
+	(footprint "LHRS_Connectors:Banana_Jack_1_Pin_4mm"
 		(layer "F.Cu")
 		(at 161.96892 76.48275)
@@
 		(embedded_fonts no)
 	)
-	(footprint "UTSVT_Connectors:Molex_Nano-Fit_105313-xx04_1x04_P2.50mm_Horizontal"
+	(footprint "LHRS_Connectors:Molex_Nano-Fit_105313-xx04_1x04_P2.50mm_Horizontal"
 		(layer "F.Cu")
 		(at 158.02 23.5)
@@
 		(descr "Plated Hole as test Point, diameter 2.0mm")
 		(tags "test point plated hole")
-		(property "Reference" "2&3"
+		(property "Reference" "TP3"
 			(at 0 -2.498 0)
 			(layer "F.SilkS")
@@
 		(descr "Plated Hole as test Point, diameter 2.0mm")
 		(tags "test point plated hole")
-		(property "Reference" "5&6"
+		(property "Reference" "TP6"
 			(at 0 -2.498 0)
 			(layer "F.SilkS")
@@
 		(descr "Plated Hole as test Point, diameter 2.0mm")
 		(tags "test point plated hole")
-		(property "Reference" "3&4"
+		(property "Reference" "TP4"
 			(at 0 -2.498 0)
 			(layer "F.SilkS")
@@
 		(descr "Plated Hole as test Point, diameter 2.0mm")
 		(tags "test point plated hole")
-		(property "Reference" "GND"
+		(property "Reference" "TP1"
 			(at 0 -2.498 0)
 			(layer "F.SilkS")
@@
 		(descr "Plated Hole as test Point, diameter 2.0mm")
 		(tags "test point plated hole")
-		(property "Reference" "7&8"
+		(property "Reference" "TP8"
 			(at 0 -2.498 0)
 			(layer "F.SilkS")
@@
 		)
 	)
-	(footprint "UTSVT_Connectors:Molex_Nano-Fit_105313-xx05_1x05_P2.50mm_Horizontal"
+	(footprint "LHRS_Connectors:Molex_Nano-Fit_105313-xx05_1x05_P2.50mm_Horizontal"
 		(layer "F.Cu")
 		(at 130.12 33.275 180)
@@
 		(tags "connector Molex Nano-Fit top entry")
 		(property "Reference" "J8"
-			(at 6.15 -2.92 0)
+			(at 6.15 -2.92 180)
 			(layer "F.SilkS")
 			(effects
@@
 		)
 		(property "Value" "therm_set2"
-			(at 6.15 12.92 0)
+			(at 6.15 12.92 180)
 			(layer "F.Fab")
 			(effects
@@
 		)
 		(fp_text user "${REFERENCE}"
-			(at 6.15 11.02 0)
+			(at 6.15 11.02 180)
 			(layer "F.Fab")
 			(effects
@@
 		(descr "Plated Hole as test Point, diameter 2.0mm")
 		(tags "test point plated hole")
-		(property "Reference" "1&2"
+		(property "Reference" "TP2"
 			(at 0 -2.498 0)
 			(layer "F.SilkS")
@@
 		)
 	)
-	(footprint "UTSVT_Connectors:Molex_Nano-Fit_105313-xx04_1x04_P2.50mm_Horizontal"
+	(footprint "LHRS_Connectors:Molex_Nano-Fit_105313-xx04_1x04_P2.50mm_Horizontal"
 		(layer "F.Cu")
 		(at 158.02 38.3)
@@
 		(descr "Plated Hole as test Point, diameter 2.0mm")
 		(tags "test point plated hole")
-		(property "Reference" "6&7"
+		(property "Reference" "TP7"
 			(at 0 -2.498 0)
 			(layer "F.SilkS")
@@
 		(embedded_fonts no)
 	)
-	(footprint "UTSVT_Connectors:Molex_Nano-Fit_105313-xx07_1x07_P2.50mm_Horizontal"
+	(footprint "LHRS_Connectors:Molex_Nano-Fit_105313-xx07_1x07_P2.50mm_Horizontal"
 		(layer "F.Cu")
 		(at 151.46892 72.38275 -90)
@@
 		(tags "connector Molex Nano-Fit top entry")
 		(property "Reference" "J1"
-			(at 6.15 -2.92 90)
+			(at 6.15 -2.92 270)
 			(layer "F.SilkS")
 			(effects
@@
 		)
 		(property "Value" "bms_taps"
-			(at 6.15 17.92 90)
+			(at 6.15 17.92 270)
 			(layer "F.Fab")
 			(effects
@@
 		)
 		(fp_text user "${REFERENCE}"
-			(at 6.15 16.02 90)
+			(at 6.15 16.02 270)
 			(layer "F.Fab")
 			(effects
@@
 		)
 	)
-	(footprint "UTSVT_Connectors:Molex_Nano-Fit_105313-xx05_1x05_P2.50mm_Horizontal"
+	(footprint "LHRS_Connectors:Molex_Nano-Fit_105313-xx05_1x05_P2.50mm_Horizontal"
 		(layer "F.Cu")
 		(at 130.14 50.575 180)
@@
 		(tags "connector Molex Nano-Fit top entry")
 		(property "Reference" "J7"
-			(at 6.15 -2.92 0)
+			(at 6.15 -2.92 180)
 			(layer "F.SilkS")
 			(effects
@@
 		)
 		(property "Value" "therm_set1"
-			(at 6.15 12.92 0)
+			(at 6.15 12.92 180)
 			(layer "F.Fab")
 			(effects
@@
 		)
 		(fp_text user "${REFERENCE}"
-			(at 6.15 11.02 0)
+			(at 6.15 11.02 180)
 			(layer "F.Fab")
 			(effects
@@
 		(descr "Plated Hole as test Point, diameter 2.0mm")
 		(tags "test point plated hole")
-		(property "Reference" "28.8[v]"
+		(property "Reference" "TP9"
 			(at 0 -2.498 0)
 			(layer "F.SilkS")
@@
 		(embedded_fonts no)
 	)
-	(footprint "UTSVT_Connectors:Banana_Jack_1_Pin_4mm"
+	(footprint "LHRS_Connectors:Banana_Jack_1_Pin_4mm"
 		(layer "F.Cu")
 		(at 126.06892 76.38275)

Commit message: images added tee hee
Parts:
- added G***: LOGO, LOGO, B.Cu at (141.8, 35.9)
- renumbered TP2 to 1&2, TP3 to 2&3, TP9 to 28.8[v], TP4 to 3&4, TP5 to 4&5, TP6 to 5&6, TP7 to 6&7, TP8 to 7&8, TP1 to GND
Other:
- board text added: "Cell Simulator Board clark rucker sep. 2026"
