File: PS-CellSim/PS-CellSim.kicad_sch (KiCad schematic)
At the start: 57 parts, among them J1 bms_taps, J2 bench_vcc, J3 bench_gnd, J4 bms_ref, J5 bms_gpio_set2, J6 bms_gpio_set1, J7 therm_set1, J8 therm_set2

Commit message: layour layouted
Parts:
- added TP1, TP2, TP3, TP4, TP5, TP6, TP7, TP8, TP9: TestPoint, TestPoint:TestPoint_Plated_Hole_D2.0mm, symbol Connector:TestPoint
Connections:
- net 1&2: now also TP2.1
- net 2&3: now also TP3.1
- net 3&4: now also TP4.1
- net 4&5: now also TP5.1
- net 5&6: now also TP6.1
- net 6&7: now also TP7.1
- net 7&8: now also TP8.1
- net GND: now also TP1.1
- net VCC: now also TP9.1
Other:
- note added: "28.8 to simulate module"

Commit message: now has kicad sharepoint smiley face :)
Parts:
- J1: footprint UTSVT_Connectors:Molex_Nano-Fit_105313-xx07_1x07_P2.50mm_Horizontal -> LHRS_Connectors:Molex_Nano-Fit_105313-xx07_1x07_P2.50mm_Horizontal
- J2, J3: footprint UTSVT_Connectors:Banana_Jack_1_Pin_4mm -> LHRS_Connectors:Banana_Jack_1_Pin_4mm
- J4: footprint UTSVT_Connectors:Molex_Nano-Fit_105313-xx02_1x02_P2.50mm_Horizontal -> LHRS_Connectors:Molex_Nano-Fit_105313-xx02_1x02_P2.50mm_Horizontal
- J5, J6: footprint UTSVT_Connectors:Molex_Nano-Fit_105313-xx04_1x04_P2.50mm_Horizontal -> LHRS_Connectors:Molex_Nano-Fit_105313-xx04_1x04_P2.50mm_Horizontal
- J7, J8: footprint UTSVT_Connectors:Molex_Nano-Fit_105313-xx05_1x05_P2.50mm_Horizontal -> LHRS_Connectors:Molex_Nano-Fit_105313-xx05_1x05_P2.50mm_Horizontal
Changed lines of the file:
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@@
 			)
 		)
-		(property "Footprint" "UTSVT_Connectors:Banana_Jack_1_Pin_4mm"
+		(property "Footprint" "LHRS_Connectors:Banana_Jack_1_Pin_4mm"
 			(at 31.75 64.77 0)
 			(hide yes)
@@
 			)
 		)
-		(property "Footprint" "UTSVT_Connectors:Molex_Nano-Fit_105313-xx04_1x04_P2.50mm_Horizontal"
+		(property "Footprint" "LHRS_Connectors:Molex_Nano-Fit_105313-xx04_1x04_P2.50mm_Horizontal"
 			(at 115.57 64.77 0)
 			(hide yes)
@@
 			)
 		)
-		(property "Footprint" "UTSVT_Connectors:Molex_Nano-Fit_105313-xx05_1x05_P2.50mm_Horizontal"
+		(property "Footprint" "LHRS_Connectors:Molex_Nano-Fit_105313-xx05_1x05_P2.50mm_Horizontal"
 			(at 147.32 45.72 0)
 			(hide yes)
@@
 			)
 		)
-		(property "Footprint" "UTSVT_Connectors:Molex_Nano-Fit_105313-xx02_1x02_P2.50mm_Horizontal"
+		(property "Footprint" "LHRS_Connectors:Molex_Nano-Fit_105313-xx02_1x02_P2.50mm_Horizontal"
 			(at 114.3 43.18 0)
 			(hide yes)
@@
 			)
 		)
-		(property "Footprint" "UTSVT_Connectors:Banana_Jack_1_Pin_4mm"
+		(property "Footprint" "LHRS_Connectors:Banana_Jack_1_Pin_4mm"
 			(at 31.75 58.42 0)
 			(hide yes)
@@
 			)
 		)
-		(property "Footprint" "UTSVT_Connectors:Molex_Nano-Fit_105313-xx05_1x05_P2.50mm_Horizontal"
+		(property "Footprint" "LHRS_Connectors:Molex_Nano-Fit_105313-xx05_1x05_P2.50mm_Horizontal"
 			(at 147.32 60.96 0)
 			(hide yes)
@@
 			)
 		)
-		(property "Footprint" "UTSVT_Connectors:Molex_Nano-Fit_105313-xx07_1x07_P2.50mm_Horizontal"
+		(property "Footprint" "LHRS_Connectors:Molex_Nano-Fit_105313-xx07_1x07_P2.50mm_Horizontal"
 			(at 30.48 91.44 0)
 			(hide yes)
@@
 			)
 		)
-		(property "Footprint" "UTSVT_Connectors:Molex_Nano-Fit_105313-xx04_1x04_P2.50mm_Horizontal"
+		(property "Footprint" "LHRS_Connectors:Molex_Nano-Fit_105313-xx04_1x04_P2.50mm_Horizontal"
 			(at 115.57 76.2 0)
 			(hide yes)

Commit message: added p/n
Parts:
- C1: P/N (none) -> CC0603KRX7R9BB105
- D1, D2, D3, D4, D5, D6, D7, D8: P/N (none) -> LTST-C193TBKT-5A
- J1: P/N (none) -> 105313-xx07
- J4: P/N (none) -> 105313-xx02
- J5, J6: P/N (none) -> 105313-xx04
- J7, J8: P/N (none) -> 105313-xx05
- R1, R2, R3, R4, R5, R6, R7, R8: value 50Ω -> 100Ω; P/N (none) -> 0603WAF1000T5E
- R10, R12, R14, R16, R18, R20, R22, R24: value 250 Ω -> 1k Ω; P/N (none) -> 0603WAF1001T5E
- R11, R13, R15, R17, R19, R21, R23, R9: P/N (none) -> 0603WAF1002T5E

Commit message: bannananana
Parts:
- J2, J3: P/N (none) -> 575-4
Changed lines of the file:
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@@
+			)
+		)
+		(property "P/N" "575-4"
+			(at 31.75 64.77 0)
+			(hide yes)
+			(show_name no)
+			(do_not_autoplace no)
+			(effects
+				(font
+					(size 1.27 1.27)
+				)
 			)
 		)
@@
 			(at 31.75 58.42 0)
 			(hide yes)
+			(show_name no)
+			(do_not_autoplace no)
+			(effects
+				(font
+					(size 1.27 1.27)
+				)
+			)
+		)
+		(property "P/N" "575-4"
+			(at 31.75 58.42 0)
+			(hide yes)
