File: hardware/.history/PS-SegmentMonitoringBoard.kicad_sch (KiCad schematic)
At the start: 16 parts, among them IC1 BQ79616PAPR, J1 voltTapsConn, J2 highSideConn, J3 lowSideConn, J4 thermsConn

Commit message: updated layout v2, everything besides silkscreen
Parts:
- removed J2: highSideConn, LHRS_Connectors:Molex_Nano-Fit_105313-xx02_1x02_P2.50mm_Horizontal, symbol Connector_Generic:Conn_01x02
- removed NT1: NetTie_4_Cross, symbol Device:NetTie_4_Cross
- added J2: highSideConn, LHRS_Connectors:Molex_Nano-Fit_105313-xx03_1x03_P2.50mm_Horizontal, symbol Connector_Generic:Conn_01x03
- added LOGO1: Dr. Hallock, LHRS_Logos:LHRs_LOGO, symbol lhrs_misc:Logo_Placeholder
- added TP7: V0, TestPoint:TestPoint_Plated_Hole_D2.0mm, symbol Connector:TestPoint
- TP6: value BAT -> V7
Connections:
- net CVSS is gone; now on net AVSS: C3.2, C4.2, C5.2, C7.1, IC1.46 (CVSS)
- net DVSS is gone; now on net AVSS: C6.2, IC1.50 (DVSS)
- net REFHM is gone; now on net AVSS: C1.2, IC1.36 (REFHM)
- net V0: now also TP7.1
- net highSideIsolation/isolatedCOMHN: now also J2.1 (Pin_1)
- net highSideIsolation/isolatedCOMHP: now also J2.2 (Pin_2)
- no-connect marks 4 -> 5
Other:
- note added: "A"
- note added: "Segment Monitoring Board"
- note removed: "Major Todo's: - redo resistor math for 240mA -> DONE - figure out NFAULT -> im p sure we dont need - double check whether I need NTC filters or not -> DONE - cap isolation with choke shi -> DONE"
- note removed: "notes n shi: - 4.7 uF - res ->"
