File: hardware/.history/lowSideIsolation.kicad_sch (KiCad schematic)
At the start: 10 parts

Commit message: layout fp updates, CB trace increases, n more
Parts:
- TR2: footprint RF_Mini-Circuits:Mini-Circuits_CD636_H4.11mm -> Custom-Footprints:SOP254P1270X685-6N
Changed lines of the file:
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@@
 			)
 		)
-		(property "Footprint" "RF_Mini-Circuits:Mini-Circuits_CD636_H4.11mm"
+		(property "Footprint" "Custom-Footprints:SOP254P1270X685-6N"
 			(at 184.15 111.76 0)
 			(hide yes)

Commit message: updated layout v2, everything besides silkscreen
Parts:
- TR2: value ADTT3-2 -> HMU1228NL
Changed lines of the file:
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@@
 			)
 		)
-		(property "Value" "ADTT3-2"
+		(property "Value" "HMU1228NL"
 			(at 184.15 129.032 0)
 			(show_name no)
