File: hardware/SMB/PS-SegmentMonitoringBoard.kicad_pcb (KiCad board)
At the start: 4 copper layers, 83.9 x 80.3 mm, 120 parts, among them IC1 BQ79616PAPR, J1 voltTapsConn, J2 highSideConn, J3 lowSideConn, J4 thermsConn, Q1 ZXTN4004KTC

Commit message: added more ss
Parts:
- added G***: LOGO, LOGO, B.Cu at (98.0, 79.8)
- moved G*** 2.44 mm to (121.6, 68.5)
- moved G*** 0.21 mm to (95.6, 129.9)
