File: hardware/SMB/PS-SegmentMonitoringBoard.kicad_sch (KiCad schematic)
At the start: 17 parts, among them IC1 BQ79616PAPR, J1 voltTapsConn, J2 highSideConn, J3 lowSideConn, J4 thermsConn

Commit message: layout v3, everything done
Parts:
- added H1, H2, H3, H4: MountingHole, MountingHole:MountingHole_3.2mm_M3, symbol Mechanical:MountingHole
